File: feedbackProject/feedbackProject.kicad_sch (KiCad schematic)
At the start: 0 parts

Commit message: library update check
Parts:
- added C1: 0,1 мк, symbol gostPassiveComponents:capacitor
- added D1: Arduino Pro Micro, symbol gostArduino:proMicro
- added DA1: AD8220, symbol gostAmplifiers:AD8220
- added DD1: L293D, symbol gostDrivers:L293D
- added R1: 3,3 к, symbol gostPassiveComponents:resistor
- added R2: 510, symbol gostPassiveComponents:resistor
- added R3: 20 к, symbol gostPassiveComponents:resistor
- added R4: 9,8 к, symbol gostPassiveComponents:resistor
- added R5: 10 к, symbol gostPassiveComponents:resistor
- added R6: 100 к, symbol gostPassiveComponents:resistor
- added VD1: BZX55C2V4, symbol gostSimpleActiveComponents:Zener_diode
- added VD2: PMEG2020, symbol gostSimpleActiveComponents:diode_Schottky
- added VT1: X, symbol gostSimpleActiveComponents:n-ch-enhancement-mosfet
- added XP1, XP2: Molex kk 254, symbol gostConnectorsAndHeaders:6pin_male_header
- added XP3: Molex kk 254, symbol gostConnectorsAndHeaders:4pin_male_header
- added XS1: USB тип C, symbol gostConnectorsAndHeaders:4pin_female_header
Connections:
- new net: D1.0, XP3.2
- new net: D1.1, XP3.3
- new net: R5.2, R6.2, VT1.1
- new net: DA1.4, R2.1, VD1.
- new net: DA1.2, XP1.2
- new net: D1.19, R3.2, XP1.4
- new net: D1.20, R4.1, XP1.6
- new net: VD2., VT1.2, XP2.5
- new net: DD1.13, XP2.1
- new net: DD1.14, XP2.2
- new net: DD1.15, XP2.3
- new net: DD1.16, XP2.4
- new net: D1.6, DD1.2
- new net: D1.7, DD1.3
- new net: D1.8, DD1.5
- new net: D1.9, DD1.6
- new net: D1.5, R5.1
- new net: DA1.6, R1.1
- new net: DA1.7, R1.2
- new net: D1.18, DA1.8
- new net +5V: C1.2, D1.13, DA1.3, DD1.1, DD1.4, DD1.7, DD1.8, R2.2, R3.1, R4.2, VD2., XP2.6, XP3.1, XS1.1
- new net GND: C1.1, D1.11, D1.12, D1.22, DA1.1, DA1.5, DD1.10, DD1.11, DD1.12, DD1.9, R6.1, VD1., VT1.3, XP1.1, XP1.3, XP1.5, XP3.4, XS1.4
Other:
- company: (none) -> МГТУ им. Н.Э. Баумана кафедра БМТ2
- title: (none) -> Схема электрическая принципиальная
