File: feedbackProject/feedbackProject.kicad_sch (KiCad schematic)
At the start: 17 parts

Commit message: some fixes + PCB
Parts:
- removed XS1: USB тип C, symbol gostConnectorsAndHeaders:4pin_female_header
- added XS1: USB тип C, MyPCBConnectorsAndHeaders:USB-Type-C-4125-GF-A-0190, symbol gostConnectorsAndHeaders:6pin_female_header
- C1: footprint (none) -> MySmdSimpleComponents:capacitor_0805_Most_Density
- D1: footprint (none) -> ArduinoPCB:proMicroSMD
- DA1: footprint (none) -> MySmdIntegratedCircuits:MSOP-8
- DD1: footprint (none) -> MyThroughHoleIntegraitedCircuits:PowerDIP-16
- R1, R2, R3, R4, R5, R6: footprint (none) -> MySmdSimpleComponents:resistor_0805_Most_Density
- VD1: footprint (none) -> MySmdSimpleComponents:diode_SOD-80C_Most_Density
- VD2: footprint (none) -> MySmdSimpleComponents:diode_SOD-323_Most_Density
- VT1: value X -> DMG1012UW-7; footprint (none) -> MySmdSimpleComponents:transistor-SOT-323
- XP1, XP2: value Molex kk 254 -> WF-6R; footprint (none) -> MyPCBConnectorsAndHeaders:WF-6R
- XP3: value Molex kk 254 -> WF-4R; footprint (none) -> MyPCBConnectorsAndHeaders:WF-4R
Connections:
- net +5V: now also DA1.8, DD1.16, DD1.9, VD2.C, XS1.2, XS1.5; no longer DA1.3, DD1.4, DD1.7, VD2.
- net GND: now also DD1.13, DD1.4, DD1.5, VD1.A, XS1.1, XS1.6; no longer DD1.10, DD1.11, DD1.9, VD1.
- net at XP1.2: now also DA1.4; no longer DA1.2
- net at R4.1, XP1.6: now also D1.18; no longer D1.20
- net at VT1.2, XP2.5: now also VD2.A; no longer VD2.
- net at XP2.1: now also DD1.11; no longer DD1.13
- net at DD1.14: now also XP2.4; no longer XP2.2
- net at DD1.15: now also D1.6; no longer XP2.3
- net at DD1.2: now also D1.7; no longer D1.6
- net at DD1.3: now also XP2.3; no longer D1.7
- net at D1.8: now also DD1.7; no longer DD1.5
- net at D1.9: now also DD1.10; no longer DD1.6
- net at DA1.6: now also R2.1, VD1.C; no longer R1.1
- net at R1.2: now also DA1.2; no longer DA1.7
- net at D1.21: now also DA1.7
- new net: DD1.6, XP2.2
- new net: DA1.3, R1.1
Other:
- moved on the sheet: R6, XP2
